File: PiInTheSky-Mainboard-v2.3.sch (EAGLE design)
At the start: 50 parts, among them Q1 MOSFET-PCHANNELSMD

Commit message: Pushed V2.3
Amended enable line on ADC
Connections:
- removed net NSS1: U$1.24-GPIO8
- net MCP3002/SDN: now also U$1.24-GPIO8; no longer U$1.27-ID_SD
Changed lines of the file:
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@@
 </segment>
 <segment>
-<pinref part="U$1" gate="G$1" pin="27-ID_SD"/>
-<wire x1="64.77" y1="-17.78" x2="54.61" y2="-17.78" width="0.1524" layer="91"/>
-<label x="54.61" y="-17.78" size="1.27" layer="95" rot="R180" xref="yes"/>
+<wire x1="113.03" y1="-7.62" x2="124.46" y2="-7.62" width="0.1524" layer="91"/>
+<label x="124.46" y="-7.62" size="1.27" layer="95" xref="yes"/>
+<pinref part="U$1" gate="G$1" pin="24-GPIO8"/>
 </segment>
 </net>
@@
 </segment>
 </net>
-<net name="NSS1" class="0">
-<segment>
-<wire x1="113.03" y1="-7.62" x2="124.46" y2="-7.62" width="0.1524" layer="91"/>
-<label x="124.46" y="-7.62" size="1.27" layer="95" xref="yes"/>
-<pinref part="U$1" gate="G$1" pin="24-GPIO8"/>
-</segment>
-</net>
